File: GPIO_board/gpio_board.sch (EAGLE design)
At the start: 15 parts, among them J1 SWITCHES, J2 LED1, J3 LED2, Q1 IRF520, Q2 IRF520, Q3 IRF520, X1 PCI-E-164SLOT

Commit message: routed some things
not final. need to finish outline and dimensions of board. need to
determine what other things need to go through the PCI connector (If
any).
Connections:
- net GND: now also X1.A10, X1.A11, X1.A8, X1.A9
- net N$11: now also U$1.6/PWM; no longer U$1.4/CAN-RX-PWM
- net N$8: now also U$1.4/CAN-RX-PWM; no longer U$1.6/PWM
- net VCC: now also J2.4, J3.4, X1.A1, X1.A2, X1.A3, X1.A4
Other:
- moved on the sheet: X1
Changed lines of the file:
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@@
 <layers>
 <layer number="1" name="Top" color="4" fill="1" visible="no" active="no"/>
+<layer number="2" name="Route2" color="1" fill="3" visible="no" active="no"/>
+<layer number="3" name="Route3" color="4" fill="3" visible="no" active="no"/>
+<layer number="4" name="Route4" color="1" fill="4" visible="no" active="no"/>
+<layer number="5" name="Route5" color="4" fill="4" visible="no" active="no"/>
+<layer number="6" name="Route6" color="1" fill="8" visible="no" active="no"/>
+<layer number="7" name="Route7" color="4" fill="8" visible="no" active="no"/>
+<layer number="8" name="Route8" color="1" fill="2" visible="no" active="no"/>
+<layer number="9" name="Route9" color="4" fill="2" visible="no" active="no"/>
+<layer number="10" name="Route10" color="1" fill="7" visible="no" active="no"/>
+<layer number="11" name="Route11" color="4" fill="7" visible="no" active="no"/>
+<layer number="12" name="Route12" color="1" fill="5" visible="no" active="no"/>
+<layer number="13" name="Route13" color="4" fill="5" visible="no" active="no"/>
+<layer number="14" name="Route14" color="1" fill="6" visible="no" active="no"/>
+<layer number="15" name="Route15" color="4" fill="6" visible="no" active="no"/>
 <layer number="16" name="Bottom" color="1" fill="1" visible="no" active="no"/>
 <layer number="17" name="Pads" color="2" fill="1" visible="no" active="no"/>
@@
 <part name="J2" library="SparkFun-Connectors" deviceset="M04" device="PTH" value="LED1"/>
 <part name="J3" library="SparkFun-Connectors" deviceset="M04" device="PTH" value="LED2"/>
-<part name="X1" library="con-pc" deviceset="PCI-E-164" device="SLOT"/>
 <part name="GND1" library="SparkFun-Aesthetics" deviceset="GND" device=""/>
 <part name="GND2" library="SparkFun-Aesthetics" deviceset="GND" device=""/>
@@
 <part name="SG1" library="SparkFun-Electromechanical" deviceset="BUZZER" device="PTH"/>
 <part name="U$2" library="talon_lbr" deviceset="PROTO_GRID" device=""/>
+<part name="X1" library="con-pc" deviceset="PCI-E-164" device="SLOT"/>
+<part name="SUPPLY1" library="SparkFun-Aesthetics" deviceset="VCC" device="" value="12V"/>
+<part name="GND4" library="SparkFun-Aesthetics" deviceset="GND" device=""/>
 </parts>
 <sheets>
@@
 <instance part="J2" gate="G$1" x="172.72" y="170.18"/>
 <instance part="J3" gate="G$1" x="195.58" y="170.18"/>
-<instance part="X1" gate="G$1" x="269.24" y="76.2"/>
 <instance part="GND1" gate="1" x="134.62" y="142.24"/>
 <instance part="GND2" gate="1" x="63.5" y="101.6"/>
@@
 <instance part="SG1" gate="G$1" x="175.26" y="104.14"/>
 <instance part="U$2" gate="G$1" x="139.7" y="50.8" rot="R270"/>
+<instance part="X1" gate="G$1" x="254" y="91.44"/>
+<instance part="SUPPLY1" gate="G$1" x="228.6" y="203.2"/>
+<instance part="GND4" gate="1" x="228.6" y="162.56"/>
 </instances>
 <busses>
@@
 <pinref part="GND1" gate="1" pin="GND"/>
 </segment>
+<segment>
+<pinref part="GND4" gate="1" pin="GND"/>
+<wire x1="228.6" y1="165.1" x2="228.6" y2="167.64" width="0.1524" layer="91"/>
+<pinref part="X1" gate="G$1" pin="A11"/>
+<wire x1="228.6" y1="167.64" x2="241.3" y2="167.64" width="0.1524" layer="91"/>
+<pinref part="X1" gate="G$1" pin="A10"/>
+<wire x1="241.3" y1="170.18" x2="228.6" y2="170.18" width="0.1524" layer="91"/>
+<wire x1="228.6" y1="170.18" x2="228.6" y2="167.64" width="0.1524" layer="91"/>
+<junction x="228.6" y="167.64"/>
+<pinref part="X1" gate="G$1" pin="A9"/>
+<wire x1="241.3" y1="172.72" x2="228.6" y2="172.72" width="0.1524" layer="91"/>
+<wire x1="228.6" y1="172.72" x2="228.6" y2="170.18" width="0.1524" layer="91"/>
+<junction x="228.6" y="170.18"/>
+<pinref part="X1" gate="G$1" pin="A8"/>
+<wire x1="241.3" y1="175.26" x2="228.6" y2="175.26" width="0.1524" layer="91"/>
+<wire x1="228.6" y1="175.26" x2="228.6" y2="172.72" width="0.1524" layer="91"/>
+<junction x="228.6" y="172.72"/>
+</segment>
 </net>
 <net name="N$1" class="0">
@@
 <wire x1="71.12" y1="129.54" x2="71.12" y2="147.32" width="0.1524" layer="91"/>
 </segment>
+<segment>
+<pinref part="X1" gate="G$1" pin="A1"/>
+<pinref part="SUPPLY1" gate="G$1" pin="VCC"/>
+<wire x1="241.3" y1="193.04" x2="228.6" y2="193.04" width="0.1524" layer="91"/>
+<wire x1="228.6" y1="193.04" x2="228.6" y2="203.2" width="0.1524" layer="91"/>
+<pinref part="X1" gate="G$1" pin="A2"/>
+<wire x1="241.3" y1="190.5" x2="228.6" y2="190.5" width="0.1524" layer="91"/>
+<wire x1="228.6" y1="190.5" x2="228.6" y2="193.04" width="0.1524" layer="91"/>
+<junction x="228.6" y="193.04"/>
+<pinref part="X1" gate="G$1" pin="A3"/>
+<wire x1="241.3" y1="187.96" x2="228.6" y2="187.96" width="0.1524" layer="91"/>
+<wire x1="228.6" y1="187.96" x2="228.6" y2="190.5" width="0.1524" layer="91"/>
+<junction x="228.6" y="190.5"/>
+<pinref part="X1" gate="G$1" pin="A4"/>
+<wire x1="241.3" y1="185.42" x2="228.6" y2="185.42" width="0.1524" layer="91"/>
+<wire x1="228.6" y1="185.42" x2="228.6" y2="187.96" width="0.1524" layer="91"/>
+<junction x="228.6" y="187.96"/>
+<pinref part="J2" gate="G$1" pin="4"/>
+<wire x1="177.8" y1="175.26" x2="182.88" y2="175.26" width="0.1524" layer="91"/>
+<wire x1="182.88" y1="175.26" x2="182.88" y2="185.42" width="0.1524" layer="91"/>
+<wire x1="182.88" y1="185.42" x2="200.66" y2="185.42" width="0.1524" layer="91"/>
+<junction x="228.6" y="185.42"/>
+<pinref part="J3" gate="G$1" pin="4"/>
+<wire x1="200.66" y1="185.42" x2="228.6" y2="185.42" width="0.1524" layer="91"/>
+<wire x1="200.66" y1="175.26" x2="200.66" y2="185.42" width="0.1524" layer="91"/>
+<junction x="200.66" y="185.42"/>
+</segment>
 </net>
 <net name="N$9" class="0">
@@
 <pinref part="R1" gate="G$1" pin="1"/>
 <wire x1="157.48" y1="132.08" x2="152.4" y2="132.08" width="0.1524" layer="91"/>
-<wire x1="152.4" y1="132.08" x2="152.4" y2="121.92" width="0.1524" layer="91"/>
-<pinref part="U$1" gate="G$1" pin="4/CAN-RX-PWM"/>
-<wire x1="152.4" y1="121.92" x2="119.38" y2="121.92" width="0.1524" layer="91"/>
+<pinref part="U$1" gate="G$1" pin="6/PWM"/>
+<wire x1="119.38" y1="116.84" x2="152.4" y2="116.84" width="0.1524" layer="91"/>
+<wire x1="152.4" y1="116.84" x2="152.4" y2="132.08" width="0.1524" layer="91"/>
 </segment>
 </net>
@@
 <segment>
 <pinref part="R3" gate="G$1" pin="1"/>
-<wire x1="157.48" y1="121.92" x2="157.48" y2="116.84" width="0.1524" layer="91"/>
-<pinref part="U$1" gate="G$1" pin="6/PWM"/>
-<wire x1="157.48" y1="116.84" x2="119.38" y2="116.84" width="0.1524" layer="91"/>
-</segment>
-</net>
+<pinref part="U$1" gate="G$1" pin="4/CAN-RX-PWM"/>
+<wire x1="119.38" y1="121.92" x2="157.48" y2="121.92" width="0.1524" layer="91"/>
+</segment>
+</net>

Commit message: routed all connections
Connections:
- net 3.3V: now also U$1.3.3V
- net VCC: no longer U$1.3.3V
Changed lines of the file:
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@@
 <part name="R4" library="SparkFun-Passives" deviceset="RESISTOR" device="EZ"/>
 <part name="R5" library="SparkFun-Passives" deviceset="RESISTOR" device="EZ"/>
-<part name="SUPPLY5" library="SparkFun-Aesthetics" deviceset="VCC" device="" value="+3.3V"/>
 <part name="SUPPLY6" library="SparkFun-Aesthetics" deviceset="3.3V" device=""/>
 <part name="SG1" library="SparkFun-Electromechanical" deviceset="BUZZER" device="PTH"/>
 <part name="U$2" library="talon_lbr" deviceset="PROTO_GRID" device=""/>
 <part name="X1" library="con-pc" deviceset="PCI-E-164" device="SLOT"/>
+<part name="GND4" library="SparkFun-Aesthetics" deviceset="GND" device=""/>
 <part name="SUPPLY1" library="SparkFun-Aesthetics" deviceset="VCC" device="" value="12V"/>
-<part name="GND4" library="SparkFun-Aesthetics" deviceset="GND" device=""/>
+<part name="SUPPLY2" library="SparkFun-Aesthetics" deviceset="3.3V" device=""/>
 </parts>
 <sheets>
@@
 <instance part="R4" gate="G$1" x="129.54" y="170.18" rot="R90"/>
 <instance part="R5" gate="G$1" x="134.62" y="170.18" rot="R90"/>
-<instance part="SUPPLY5" gate="G$1" x="71.12" y="147.32"/>
 <instance part="SUPPLY6" gate="G$1" x="132.08" y="180.34"/>
 <instance part="SG1" gate="G$1" x="175.26" y="104.14"/>
 <instance part="U$2" gate="G$1" x="139.7" y="50.8" rot="R270"/>
 <instance part="X1" gate="G$1" x="254" y="91.44"/>
-<instance part="SUPPLY1" gate="G$1" x="228.6" y="203.2"/>
 <instance part="GND4" gate="1" x="228.6" y="162.56"/>
+<instance part="SUPPLY1" gate="G$1" x="223.52" y="200.66"/>
+<instance part="SUPPLY2" gate="G$1" x="68.58" y="144.78"/>
 </instances>
 <busses>
@@
 <net name="VCC" class="0">
 <segment>
-<pinref part="U$1" gate="G$1" pin="3.3V"/>
-<wire x1="73.66" y1="129.54" x2="71.12" y2="129.54" width="0.1524" layer="91"/>
-<pinref part="SUPPLY5" gate="G$1" pin="VCC"/>
-<wire x1="71.12" y1="129.54" x2="71.12" y2="147.32" width="0.1524" layer="91"/>
-</segment>
-<segment>
+<pinref part="SUPPLY1" gate="G$1" pin="VCC"/>
+<wire x1="223.52" y1="200.66" x2="223.52" y2="193.04" width="0.1524" layer="91"/>
 <pinref part="X1" gate="G$1" pin="A1"/>
-<pinref part="SUPPLY1" gate="G$1" pin="VCC"/>
 <wire x1="241.3" y1="193.04" x2="228.6" y2="193.04" width="0.1524" layer="91"/>
-<wire x1="228.6" y1="193.04" x2="228.6" y2="203.2" width="0.1524" layer="91"/>
 <pinref part="X1" gate="G$1" pin="A2"/>
 <wire x1="241.3" y1="190.5" x2="228.6" y2="190.5" width="0.1524" layer="91"/>
 <wire x1="228.6" y1="190.5" x2="228.6" y2="193.04" width="0.1524" layer="91"/>
-<junction x="228.6" y="193.04"/>
 <pinref part="X1" gate="G$1" pin="A3"/>
 <wire x1="241.3" y1="187.96" x2="228.6" y2="187.96" width="0.1524" layer="91"/>
@@
 <wire x1="200.66" y1="175.26" x2="200.66" y2="185.42" width="0.1524" layer="91"/>
 <junction x="200.66" y="185.42"/>
+<wire x1="223.52" y1="193.04" x2="228.6" y2="193.04" width="0.1524" layer="91"/>
+<junction x="228.6" y="193.04"/>
 </segment>
 </net>
@@
 <junction x="132.08" y="177.8"/>
 </segment>
-</net>
+<segment>
+<pinref part="U$1" gate="G$1" pin="3.3V"/>
+<pinref part="SUPPLY2" gate="G$1" pin="3.3V"/>
+<wire x1="73.66" y1="129.54" x2="68.58" y2="129.54" width="0.1524" layer="91"/>
+<wire x1="68.58" y1="129.54" x2="68.58" y2="144.78" width="0.1524" layer="91"/>
+</segment>
+</net>
