File: GPIO_board/gpio_board.brd (EAGLE design)
At the start: 93.6 x 79 mm, 15 parts, among them J1 SWITCHES, J2 LED1, J3 LED2, Q1 IRF520, Q2 IRF520, Q3 IRF520, X1 PCI-E-164SLOT

Commit message: routed some wires
Routing:
- net N$11: track 0.00 -> 51.5 mm
- net N$5: track 0.00 -> 46.4 mm
- net N$7: track 0.00 -> 43.3 mm
- net N$9: track 0.00 -> 38.3 mm
- net N$4: track 0.00 -> 33.6 mm, vias 0 -> 2
- net 3.3V: track 0.00 -> 32.7 mm
- net N$10: track 0.00 -> 31.6 mm
- net N$6: track 0.00 -> 31.4 mm
- net N$8: track 0.00 -> 25.3 mm
- net VCC: track 0.00 -> 22.4 mm
Changed lines of the file:
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@@
 <contactref element="Q1" pad="D"/>
 <contactref element="J3" pad="1"/>
-<wire x1="58.42" y1="69.85" x2="55.88" y2="80.01" width="0" layer="19" extent="1-1"/>
-<wire x1="35.56" y1="80.01" x2="55.88" y2="80.01" width="0" layer="19" extent="1-1"/>
+<wire x1="55.88" y1="80.01" x2="55.88" y2="77.47" width="0.4064" layer="1"/>
+<wire x1="55.88" y1="77.47" x2="58.42" y2="74.93" width="0.4064" layer="1"/>
+<wire x1="58.42" y1="74.93" x2="58.42" y2="69.85" width="0.4064" layer="1"/>
+<wire x1="35.56" y1="80.01" x2="43.18" y2="80.01" width="0.4064" layer="1"/>
+<wire x1="43.18" y1="80.01" x2="46.99" y2="76.2" width="0.4064" layer="1"/>
+<via x="46.99" y="76.2" extent="1-16" drill="0.508"/>
+<wire x1="46.99" y1="76.2" x2="53.34" y2="76.2" width="0.4064" layer="16"/>
+<wire x1="53.34" y1="76.2" x2="54.61" y2="77.47" width="0.4064" layer="16"/>
+<via x="54.61" y="77.47" extent="1-16" drill="0.508"/>
+<wire x1="54.61" y1="77.47" x2="55.88" y2="77.47" width="0.4064" layer="1"/>
 </signal>
 <signal name="N$6">
@@
 <contactref element="Q2" pad="D"/>
 <contactref element="J3" pad="2"/>
-<wire x1="46.99" y1="69.85" x2="53.34" y2="80.01" width="0" layer="19" extent="1-1"/>
-<wire x1="33.02" y1="80.01" x2="46.99" y2="69.85" width="0" layer="19" extent="1-1"/>
+<wire x1="33.02" y1="80.01" x2="33.02" y2="77.47" width="0.4064" layer="1"/>
+<wire x1="33.02" y1="77.47" x2="36.83" y2="73.66" width="0.4064" layer="1"/>
+<wire x1="36.83" y1="73.66" x2="45.72" y2="73.66" width="0.4064" layer="1"/>
+<wire x1="45.72" y1="73.66" x2="46.99" y2="72.39" width="0.4064" layer="1"/>
+<wire x1="46.99" y1="72.39" x2="46.99" y2="69.85" width="0.4064" layer="1"/>
+<wire x1="53.34" y1="80.01" x2="53.34" y2="78.74" width="0.4064" layer="1"/>
+<wire x1="53.34" y1="78.74" x2="46.99" y2="72.39" width="0.4064" layer="1"/>
 </signal>
 <signal name="N$10">
@@
 <contactref element="J2" pad="3"/>
 <contactref element="Q3" pad="D"/>
-<wire x1="34.29" y1="69.85" x2="50.8" y2="80.01" width="0" layer="19" extent="1-1"/>
-<wire x1="30.48" y1="80.01" x2="34.29" y2="69.85" width="0" layer="19" extent="1-1"/>
+<wire x1="30.48" y1="80.01" x2="30.48" y2="77.47" width="0.4064" layer="16"/>
+<wire x1="30.48" y1="77.47" x2="34.29" y2="73.66" width="0.4064" layer="16"/>
+<wire x1="34.29" y1="73.66" x2="34.29" y2="69.85" width="0.4064" layer="16"/>
+<wire x1="50.8" y1="80.01" x2="50.8" y2="78.74" width="0.4064" layer="16"/>
+<wire x1="50.8" y1="78.74" x2="49.53" y2="77.47" width="0.4064" layer="16"/>
+<wire x1="49.53" y1="77.47" x2="38.1" y2="77.47" width="0.4064" layer="16"/>
+<wire x1="38.1" y1="77.47" x2="34.29" y2="73.66" width="0.4064" layer="16"/>
 </signal>
 <signal name="VCC">
@@
 <contactref element="J2" pad="4"/>
 <contactref element="J3" pad="4"/>
-<wire x1="27.94" y1="80.01" x2="48.26" y2="80.01" width="0" layer="19" extent="1-1"/>
+<wire x1="48.26" y1="80.01" x2="45.72" y2="82.55" width="0.4064" layer="1"/>
+<wire x1="45.72" y1="82.55" x2="30.48" y2="82.55" width="0.4064" layer="1"/>
+<wire x1="30.48" y1="82.55" x2="27.94" y2="80.01" width="0.4064" layer="1"/>
 <wire x1="11.5" y1="3.75" x2="27.94" y2="80.01" width="0" layer="19" extent="16-16"/>
 <wire x1="10.5" y1="3.75" x2="11.5" y2="3.75" width="0" layer="19" extent="16-16"/>
@@
 <contactref element="R2" pad="P$1"/>
 <contactref element="U$1" pad="5"/>
-<wire x1="21.59" y1="35.56" x2="44.45" y2="58.42" width="0" layer="19" extent="1-1"/>
+<wire x1="21.59" y1="35.56" x2="27.94" y2="41.91" width="0.4064" layer="1"/>
+<wire x1="27.94" y1="41.91" x2="27.94" y2="52.07" width="0.4064" layer="1"/>
+<wire x1="27.94" y1="52.07" x2="34.29" y2="58.42" width="0.4064" layer="1"/>
+<wire x1="34.29" y1="58.42" x2="44.45" y2="58.42" width="0.4064" layer="1"/>
 </signal>
 <signal name="N$11">
 <contactref element="R1" pad="P$1"/>
 <contactref element="U$1" pad="6"/>
-<wire x1="21.59" y1="33.02" x2="55.88" y2="58.42" width="0" layer="19" extent="1-1"/>
+<wire x1="21.59" y1="33.02" x2="24.13" y2="35.56" width="0.4064" layer="1"/>
+<wire x1="24.13" y1="35.56" x2="24.13" y2="36.83" width="0.4064" layer="1"/>
+<wire x1="24.13" y1="36.83" x2="29.21" y2="41.91" width="0.4064" layer="1"/>
+<wire x1="29.21" y1="41.91" x2="29.21" y2="52.07" width="0.4064" layer="1"/>
+<wire x1="29.21" y1="52.07" x2="33.02" y2="55.88" width="0.4064" layer="1"/>
+<wire x1="33.02" y1="55.88" x2="44.45" y2="55.88" width="0.4064" layer="1"/>
+<wire x1="44.45" y1="55.88" x2="46.99" y2="58.42" width="0.4064" layer="1"/>
+<wire x1="46.99" y1="58.42" x2="55.88" y2="58.42" width="0.4064" layer="1"/>
 </signal>
 <signal name="3.3V">
@@
 <contactref element="R5" pad="P$2"/>
 <contactref element="U$1" pad="3.3V"/>
-<wire x1="16.51" y1="60.96" x2="36.83" y2="45.72" width="0" layer="19" extent="1-1"/>
-<wire x1="12.7" y1="60.96" x2="16.51" y2="60.96" width="0" layer="19" extent="1-1"/>
+<wire x1="12.7" y1="60.96" x2="16.51" y2="60.96" width="0.4064" layer="1"/>
+<wire x1="16.51" y1="60.96" x2="25.4" y2="60.96" width="0.4064" layer="16"/>
+<wire x1="25.4" y1="60.96" x2="31.75" y2="54.61" width="0.4064" layer="16"/>
+<wire x1="31.75" y1="54.61" x2="31.75" y2="50.8" width="0.4064" layer="16"/>
+<wire x1="31.75" y1="50.8" x2="36.83" y2="45.72" width="0.4064" layer="16"/>
 </signal>
 <signal name="N$5">
@@
 <contactref element="R5" pad="P$1"/>
 <contactref element="U$1" pad="2"/>
-<wire x1="12.7" y1="68.58" x2="16.51" y2="80.01" width="0" layer="19" extent="1-1"/>
-<wire x1="21.59" y1="43.18" x2="12.7" y2="68.58" width="0" layer="19" extent="1-1"/>
+<wire x1="12.7" y1="68.58" x2="15.24" y2="71.12" width="0.4064" layer="1"/>
+<wire x1="15.24" y1="71.12" x2="15.24" y2="78.74" width="0.4064" layer="1"/>
+<wire x1="15.24" y1="78.74" x2="16.51" y2="80.01" width="0.4064" layer="1"/>
+<wire x1="21.59" y1="43.18" x2="17.78" y2="43.18" width="0.4064" layer="16"/>
+<wire x1="17.78" y1="43.18" x2="16.51" y2="44.45" width="0.4064" layer="16"/>
+<wire x1="16.51" y1="44.45" x2="16.51" y2="49.53" width="0.4064" layer="16"/>
+<wire x1="16.51" y1="49.53" x2="10.16" y2="55.88" width="0.4064" layer="16"/>
+<wire x1="10.16" y1="55.88" x2="10.16" y2="66.04" width="0.4064" layer="16"/>
+<wire x1="10.16" y1="66.04" x2="12.7" y2="68.58" width="0.4064" layer="16"/>
 </signal>
 <signal name="N$7">
@@
 <contactref element="J1" pad="2"/>
 <contactref element="U$1" pad="3"/>
-<wire x1="16.51" y1="68.58" x2="19.05" y2="80.01" width="0" layer="19" extent="1-1"/>
-<wire x1="21.59" y1="40.64" x2="16.51" y2="68.58" width="0" layer="19" extent="1-1"/>
+<wire x1="16.51" y1="68.58" x2="16.51" y2="77.47" width="0.4064" layer="1"/>
+<wire x1="16.51" y1="77.47" x2="19.05" y2="80.01" width="0.4064" layer="1"/>
+<wire x1="16.51" y1="68.58" x2="17.78" y2="67.31" width="0.4064" layer="1"/>
+<wire x1="17.78" y1="67.31" x2="17.78" y2="63.5" width="0.4064" layer="1"/>
+<wire x1="17.78" y1="63.5" x2="19.05" y2="62.23" width="0.4064" layer="1"/>
+<wire x1="19.05" y1="62.23" x2="19.05" y2="41.91" width="0.4064" layer="1"/>
+<wire x1="19.05" y1="41.91" x2="20.32" y2="40.64" width="0.4064" layer="1"/>
+<wire x1="20.32" y1="40.64" x2="21.59" y2="40.64" width="0.4064" layer="1"/>
 </signal>
 <signal name="N$12">
@@
 <contactref element="R3" pad="P$1"/>
 <contactref element="U$1" pad="4"/>
-<wire x1="21.59" y1="38.1" x2="31.75" y2="58.42" width="0" layer="19" extent="1-1"/>
+<wire x1="21.59" y1="38.1" x2="22.86" y2="38.1" width="0.4064" layer="1"/>
+<wire x1="22.86" y1="38.1" x2="26.67" y2="41.91" width="0.4064" layer="1"/>
+<wire x1="26.67" y1="41.91" x2="26.67" y2="53.34" width="0.4064" layer="1"/>
+<wire x1="26.67" y1="53.34" x2="31.75" y2="58.42" width="0.4064" layer="1"/>
 </signal>
 <signal name="N$14">

Commit message: SUCCESSfully made two ground pours
Routing:
- net VCC: track 22.4 -> 132.8 mm
- net GND: track 0.00 -> 77.5 mm, vias 0 -> 2
- net N$12: track 0.00 -> 23.9 mm
- added copper zone on layer 1, net GND
Changed lines of the file:
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@@
 <vertex x="-1.27" y="83.82"/>
 </polygon>
-<wire x1="17.5" y1="3.75" x2="18.5" y2="3.75" width="0" layer="19" extent="16-16"/>
-<wire x1="16.5" y1="3.75" x2="17.5" y2="3.75" width="0" layer="19" extent="16-16"/>
-<wire x1="15.5" y1="3.75" x2="16.5" y2="3.75" width="0" layer="19" extent="16-16"/>
-<wire x1="21.59" y1="50.8" x2="18.5" y2="3.75" width="0" layer="19" extent="16-16"/>
+<wire x1="18.5" y1="3.75" x2="18.5" y2="12.7" width="0.4064" layer="16"/>
+<wire x1="18.5" y1="12.7" x2="18.5" y2="27.22" width="0.4064" layer="16"/>
+<wire x1="18.5" y1="27.22" x2="15.24" y2="30.48" width="0.4064" layer="16"/>
+<wire x1="15.24" y1="30.48" x2="15.24" y2="43.18" width="0.4064" layer="16"/>
+<via x="15.24" y="43.18" extent="1-16" drill="0.508"/>
+<wire x1="15.24" y1="43.18" x2="15.24" y2="44.45" width="0.4064" layer="1"/>
+<wire x1="15.24" y1="44.45" x2="17.78" y2="46.99" width="0.4064" layer="1"/>
+<via x="17.78" y="46.99" extent="1-16" drill="0.508"/>
+<wire x1="17.78" y1="46.99" x2="21.59" y2="50.8" width="0.4064" layer="16"/>
+<wire x1="17.5" y1="3.75" x2="17.5" y2="11.7" width="0.4064" layer="16"/>
+<wire x1="17.5" y1="11.7" x2="18.14" y2="12.34" width="0.4064" layer="16"/>
+<wire x1="18.14" y1="12.34" x2="18.5" y2="12.7" width="0.4064" layer="16"/>
+<wire x1="16.5" y1="3.75" x2="16.5" y2="10.7" width="0.4064" layer="16"/>
+<wire x1="16.5" y1="10.7" x2="17.5" y2="11.7" width="0.4064" layer="16"/>
+<wire x1="15.5" y1="3.75" x2="15.5" y2="9.7" width="0.4064" layer="16"/>
+<wire x1="15.5" y1="9.7" x2="17.5" y2="11.7" width="0.4064" layer="16"/>
+<polygon width="0.4064" layer="1">
+<vertex x="-1.27" y="83.82"/>
+<vertex x="93.98" y="83.82"/>
+<vertex x="93.98" y="7.62"/>
+<vertex x="7.62" y="7.62"/>
+<vertex x="7.62" y="8.89"/>
+<vertex x="7.62" y="11.43"/>
+<vertex x="-1.27" y="11.43"/>
+</polygon>
 </signal>
 <signal name="N$1">
@@
 <wire x1="45.72" y1="82.55" x2="30.48" y2="82.55" width="0.4064" layer="1"/>
 <wire x1="30.48" y1="82.55" x2="27.94" y2="80.01" width="0.4064" layer="1"/>
-<wire x1="11.5" y1="3.75" x2="27.94" y2="80.01" width="0" layer="19" extent="16-16"/>
-<wire x1="10.5" y1="3.75" x2="11.5" y2="3.75" width="0" layer="19" extent="16-16"/>
-<wire x1="9.5" y1="3.75" x2="10.5" y2="3.75" width="0" layer="19" extent="16-16"/>
-<wire x1="8.5" y1="3.75" x2="9.5" y2="3.75" width="0" layer="19" extent="16-16"/>
+<wire x1="27.94" y1="80.01" x2="22.86" y2="74.93" width="0.4064" layer="16"/>
+<wire x1="22.86" y1="74.93" x2="17.78" y2="74.93" width="0.4064" layer="16"/>
+<wire x1="17.78" y1="74.93" x2="5.08" y2="62.23" width="0.4064" layer="16"/>
+<wire x1="5.08" y1="62.23" x2="5.08" y2="24.13" width="0.4064" layer="16"/>
+<wire x1="5.08" y1="24.13" x2="11.43" y2="17.78" width="0.4064" layer="16"/>
+<wire x1="11.43" y1="17.78" x2="11.43" y2="10.16" width="0.4064" layer="16"/>
+<wire x1="11.43" y1="10.16" x2="11.43" y2="3.82" width="0.4064" layer="16"/>
+<wire x1="11.43" y1="3.82" x2="11.5" y2="3.75" width="0.4064" layer="16"/>
+<wire x1="10.5" y1="3.75" x2="10.5" y2="9.23" width="0.4064" layer="16"/>
+<wire x1="10.5" y1="9.23" x2="11.43" y2="10.16" width="0.4064" layer="16"/>
+<wire x1="9.5" y1="3.75" x2="9.5" y2="8.23" width="0.4064" layer="16"/>
+<wire x1="9.5" y1="8.23" x2="10.5" y2="9.23" width="0.4064" layer="16"/>
+<wire x1="8.5" y1="3.75" x2="8.5" y2="7.23" width="0.4064" layer="16"/>
+<wire x1="8.5" y1="7.23" x2="10.5" y2="9.23" width="0.4064" layer="16"/>
 </signal>
 <signal name="N$9">
@@
 <contactref element="SG1" pad="+"/>
 <contactref element="U$1" pad="7"/>
-<wire x1="21.59" y1="30.48" x2="8.89" y2="45.01" width="0" layer="19" extent="1-1"/>
+<wire x1="21.59" y1="30.48" x2="19.05" y2="30.48" width="0.4064" layer="1"/>
+<wire x1="19.05" y1="30.48" x2="17.78" y2="31.75" width="0.4064" layer="1"/>
+<wire x1="17.78" y1="31.75" x2="17.78" y2="40.64" width="0.4064" layer="1"/>
+<wire x1="17.78" y1="40.64" x2="16.51" y2="41.91" width="0.4064" layer="1"/>
+<wire x1="16.51" y1="41.91" x2="11.99" y2="41.91" width="0.4064" layer="1"/>
+<wire x1="11.99" y1="41.91" x2="8.89" y2="45.01" width="0.4064" layer="1"/>
 </signal>
 <signal name="N$8">

Commit message: connected a bunch of things to a bunch of things
Parts:
- moved U$2 109.1 mm to (0.00, -41.9), flipped to the top, turned to 0 degrees
Connections:
- new net N$29: U$2.P$32, X1.A40
- new net N$30: U$2.P$48, X1.A41
- new net N$31: U$2.P$64, X1.A42
- new net N$32: U$2.P$80, X1.A43
- new net N$33: U$2.P$96, X1.A44
- new net N$34: U$2.P$112, X1.A45
- new net N$35: U$2.P$128, X1.A46
- new net N$36: U$2.P$144, X1.A47
- new net N$37: U$2.P$160, X1.A48
- new net N$38: U$2.P$176, X1.A49
- new net N$39: U$2.P$192, X1.A50
- new net N$40: U$2.P$208, X1.A51
- new net N$41: U$2.P$224, X1.A52
- new net N$42: U$2.P$240, X1.A53
- new net N$43: U$2.P$256, X1.A54
Routing:
- net N$13: track 45.2 -> 29.0 mm
- net N$24: track 18.7 -> 2.54 mm
- net N$23: track 18.7 -> 2.54 mm
- net N$22: track 18.7 -> 2.54 mm
- net N$21: track 18.7 -> 2.54 mm
- net N$18: track 18.7 -> 2.54 mm
- net N$17: track 18.7 -> 2.54 mm
- net N$16: track 18.7 -> 2.54 mm
- net N$15: track 18.7 -> 2.54 mm
- net N$14: track 18.7 -> 2.54 mm
- net N$20: track 18.7 -> 2.54 mm
- net N$19: track 18.7 -> 2.54 mm
- net N$25: track 42.6 -> 28.2 mm
- net N$26: track 40.1 -> 27.5 mm
- net N$27: track 37.5 -> 26.8 mm
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