File: GPIO_board/gpio_board.brd (EAGLE design)
At the start: 93.6 x 79 mm, 15 parts, among them J1 SWITCHES, J2 LED1, J3 LED2, Q1 IRF520, Q2 IRF520, Q3 IRF520, X1 PCI-E-164SLOT

Commit message: something has gone horribly wrong.
assuming that all the pads in the PROTO_GRID package where placed
perfectly chronologically has resulted in a tragic waste of 30 minutes.
Apparently I couldn't just assume the entire bottom row was multiples of
16. :-1:
Parts:
- moved U$2 105.1 mm to (47.0, 52.1), flipped to the bottom, turned to 180 degrees
Changed lines of the file:
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@@
 <element name="SG1" library="SparkFun-Electromechanical" package="BUZZER-12MM" value="BUZZERPTH" x="8.89" y="48.26" rot="R270"/>
 <element name="X1" library="con-pc" package="PCI-E_SLOT" value="PCI-E-164SLOT" x="0" y="0"/>
-<element name="U$2" library="talon_lbr" package="PROTO_GRID16" value="PROTO_GRID" x="0" y="-41.91"/>
+<element name="U$2" library="talon_lbr" package="PROTO_GRID16" value="PROTO_GRID" x="46.99" y="52.07" rot="MR180"/>
 </elements>
 <signals>
@@
 <wire x1="36.83" y1="43.18" x2="39.37" y2="43.18" width="0.4064" layer="1"/>
 <contactref element="U$2" pad="P$16"/>
-<wire x1="0" y1="-41.91" x2="36.83" y2="43.18" width="0" layer="19" extent="1-1"/>
+<wire x1="46.99" y1="52.07" x2="36.83" y2="43.18" width="0" layer="19" extent="1-1"/>
 </signal>
 <signal name="N$15">
@@
 <wire x1="36.83" y1="40.64" x2="39.37" y2="40.64" width="0.4064" layer="1"/>
 <contactref element="U$2" pad="P$15"/>
-<wire x1="0" y1="-39.37" x2="36.83" y2="40.64" width="0" layer="19" extent="1-1"/>
+<wire x1="46.99" y1="49.53" x2="36.83" y2="40.64" width="0" layer="19" extent="1-1"/>
 </signal>
 <signal name="N$16">
@@
 <wire x1="36.83" y1="38.1" x2="39.37" y2="38.1" width="0.4064" layer="1"/>
 <contactref element="U$2" pad="P$14"/>
-<wire x1="0" y1="-36.83" x2="36.83" y2="38.1" width="0" layer="19" extent="1-1"/>
+<wire x1="46.99" y1="46.99" x2="36.83" y2="38.1" width="0" layer="19" extent="1-1"/>
 </signal>
 <signal name="N$17">
@@
 <wire x1="36.83" y1="35.56" x2="39.37" y2="35.56" width="0.4064" layer="1"/>
 <contactref element="U$2" pad="P$13"/>
-<wire x1="0" y1="-34.29" x2="36.83" y2="35.56" width="0" layer="19" extent="1-1"/>
+<wire x1="46.99" y1="44.45" x2="36.83" y2="35.56" width="0" layer="19" extent="1-1"/>
 </signal>
 <signal name="N$18">
@@
 <wire x1="36.83" y1="33.02" x2="39.37" y2="33.02" width="0.4064" layer="1"/>
 <contactref element="U$2" pad="P$12"/>
-<wire x1="0" y1="-31.75" x2="36.83" y2="33.02" width="0" layer="19" extent="1-1"/>
+<wire x1="46.99" y1="41.91" x2="36.83" y2="33.02" width="0" layer="19" extent="1-1"/>
 </signal>
 <signal name="N$19">
@@
 <wire x1="36.83" y1="30.48" x2="39.37" y2="30.48" width="0.4064" layer="1"/>
 <contactref element="U$2" pad="P$11"/>
-<wire x1="0" y1="-29.21" x2="36.83" y2="30.48" width="0" layer="19" extent="1-1"/>
+<wire x1="46.99" y1="39.37" x2="36.83" y2="30.48" width="0" layer="19" extent="1-1"/>
 </signal>
 <signal name="N$20">
@@
 <wire x1="36.83" y1="27.94" x2="39.37" y2="27.94" width="0.4064" layer="1"/>
 <contactref element="U$2" pad="P$10"/>
-<wire x1="0" y1="-26.67" x2="36.83" y2="27.94" width="0" layer="19" extent="1-1"/>
+<wire x1="46.99" y1="36.83" x2="36.83" y2="27.94" width="0" layer="19" extent="1-1"/>
 </signal>
 <signal name="N$21">
@@
 <wire x1="36.83" y1="25.4" x2="39.37" y2="25.4" width="0.4064" layer="1"/>
 <contactref element="U$2" pad="P$9"/>
-<wire x1="0" y1="-24.13" x2="36.83" y2="25.4" width="0" layer="19" extent="1-1"/>
+<wire x1="46.99" y1="34.29" x2="36.83" y2="25.4" width="0" layer="19" extent="1-1"/>
 </signal>
 <signal name="N$22">
@@
 <wire x1="36.83" y1="22.86" x2="39.37" y2="22.86" width="0.4064" layer="1"/>
 <contactref element="U$2" pad="P$8"/>
-<wire x1="0" y1="-21.59" x2="36.83" y2="22.86" width="0" layer="19" extent="1-1"/>
+<wire x1="46.99" y1="31.75" x2="36.83" y2="22.86" width="0" layer="19" extent="1-1"/>
 </signal>
 <signal name="N$23">
@@
 <wire x1="36.83" y1="20.32" x2="39.37" y2="20.32" width="0.4064" layer="1"/>
 <contactref element="U$2" pad="P$7"/>
-<wire x1="0" y1="-19.05" x2="36.83" y2="20.32" width="0" layer="19" extent="1-1"/>
+<wire x1="46.99" y1="29.21" x2="36.83" y2="20.32" width="0" layer="19" extent="1-1"/>
 </signal>
 <signal name="N$24">
@@
 <wire x1="36.83" y1="17.78" x2="39.37" y2="17.78" width="0.4064" layer="1"/>
 <contactref element="U$2" pad="P$6"/>
-<wire x1="0" y1="-16.51" x2="36.83" y2="17.78" width="0" layer="19" extent="1-1"/>
+<wire x1="46.99" y1="26.67" x2="36.83" y2="17.78" width="0" layer="19" extent="1-1"/>
 </signal>
 <signal name="N$13">
@@
 <wire x1="35.56" y1="15.24" x2="39.37" y2="15.24" width="0.4064" layer="1"/>
 <contactref element="U$2" pad="P$5"/>
-<wire x1="0" y1="-13.97" x2="34.29" y2="16.51" width="0" layer="19" extent="1-1"/>
+<wire x1="46.99" y1="24.13" x2="34.29" y2="16.51" width="0" layer="19" extent="1-1"/>
 </signal>
 <signal name="N$25">
@@
 <wire x1="35.56" y1="13.97" x2="40.64" y2="13.97" width="0.4064" layer="1"/>
 <contactref element="U$2" pad="P$4"/>
-<wire x1="0" y1="-11.43" x2="21.59" y2="25.4" width="0" layer="19" extent="1-1"/>
+<wire x1="46.99" y1="21.59" x2="21.59" y2="25.4" width="0" layer="19" extent="1-1"/>
 </signal>
 <signal name="N$26">
@@
 <wire x1="35.56" y1="12.7" x2="41.91" y2="12.7" width="0.4064" layer="1"/>
 <contactref element="U$2" pad="P$3"/>
-<wire x1="0" y1="-8.89" x2="21.59" y2="22.86" width="0" layer="19" extent="1-1"/>
+<wire x1="46.99" y1="19.05" x2="21.59" y2="22.86" width="0" layer="19" extent="1-1"/>
 </signal>
 <signal name="N$27">
@@
 <wire x1="35.56" y1="11.43" x2="43.18" y2="11.43" width="0.4064" layer="1"/>
 <contactref element="U$2" pad="P$2"/>
-<wire x1="0" y1="-6.35" x2="21.59" y2="20.32" width="0" layer="19" extent="1-1"/>
+<wire x1="46.99" y1="16.51" x2="21.59" y2="20.32" width="0" layer="19" extent="1-1"/>
 </signal>
 <signal name="N$28">
@@
 <wire x1="35.56" y1="10.16" x2="44.45" y2="10.16" width="0.4064" layer="1"/>
 <contactref element="U$2" pad="P$1"/>
-<wire x1="0" y1="-3.81" x2="21.59" y2="17.78" width="0" layer="19" extent="1-1"/>
+<wire x1="46.99" y1="13.97" x2="21.59" y2="17.78" width="0" layer="19" extent="1-1"/>
 </signal>
 <signal name="N$29">
 <contactref element="X1" pad="A40"/>
 <contactref element="U$2" pad="P$32"/>
-<wire x1="2.54" y1="-24.13" x2="49.5" y2="3.75" width="0" layer="19" extent="16-16"/>
+<wire x1="49.53" y1="34.29" x2="49.5" y2="3.75" width="0" layer="19" extent="16-16"/>
 </signal>
 <signal name="N$30">
 <contactref element="X1" pad="A41"/>
 <contactref element="U$2" pad="P$48"/>
-<wire x1="5.08" y1="-21.59" x2="50.5" y2="3.75" width="0" layer="19" extent="16-16"/>
+<wire x1="52.07" y1="31.75" x2="50.5" y2="3.75" width="0" layer="19" extent="16-16"/>
 </signal>
 <signal name="N$31">
 <contactref element="X1" pad="A42"/>
 <contactref element="U$2" pad="P$64"/>
-<wire x1="7.62" y1="-24.13" x2="51.5" y2="3.75" width="0" layer="19" extent="16-16"/>
+<wire x1="54.61" y1="34.29" x2="51.5" y2="3.75" width="0" layer="19" extent="16-16"/>
 </signal>
 <signal name="N$32">
 <contactref element="X1" pad="A43"/>
 <contactref element="U$2" pad="P$80"/>
-<wire x1="10.16" y1="-21.59" x2="52.5" y2="3.75" width="0" layer="19" extent="16-16"/>
+<wire x1="57.15" y1="31.75" x2="52.5" y2="3.75" width="0" layer="19" extent="16-16"/>
 </signal>
 <signal name="N$33">
 <contactref element="X1" pad="A44"/>
 <contactref element="U$2" pad="P$96"/>
-<wire x1="12.7" y1="-24.13" x2="53.5" y2="3.75" width="0" layer="19" extent="16-16"/>
+<wire x1="59.69" y1="34.29" x2="53.5" y2="3.75" width="0" layer="19" extent="16-16"/>
 </signal>
 <signal name="N$34">
 <contactref element="X1" pad="A45"/>
 <contactref element="U$2" pad="P$112"/>
-<wire x1="15.24" y1="-21.59" x2="54.5" y2="3.75" width="0" layer="19" extent="16-16"/>
+<wire x1="62.23" y1="31.75" x2="54.5" y2="3.75" width="0" layer="19" extent="16-16"/>
 </signal>
 <signal name="N$35">
 <contactref element="X1" pad="A46"/>
 <contactref element="U$2" pad="P$128"/>
-<wire x1="17.78" y1="-24.13" x2="55.5" y2="3.75" width="0" layer="19" extent="16-16"/>
+<wire x1="64.77" y1="34.29" x2="55.5" y2="3.75" width="0" layer="19" extent="16-16"/>
 </signal>
 <signal name="N$36">
 <contactref element="X1" pad="A47"/>
 <contactref element="U$2" pad="P$144"/>
-<wire x1="20.32" y1="-21.59" x2="56.5" y2="3.75" width="0" layer="19" extent="16-16"/>
+<wire x1="67.31" y1="31.75" x2="56.5" y2="3.75" width="0" layer="19" extent="16-16"/>
 </signal>
 <signal name="N$37">
 <contactref element="X1" pad="A48"/>
 <contactref element="U$2" pad="P$160"/>
-<wire x1="22.86" y1="-24.13" x2="57.5" y2="3.75" width="0" layer="19" extent="16-16"/>
+<wire x1="69.85" y1="34.29" x2="57.5" y2="3.75" width="0" layer="19" extent="16-16"/>
 </signal>
 <signal name="N$38">
 <contactref element="X1" pad="A49"/>
 <contactref element="U$2" pad="P$176"/>
-<wire x1="25.4" y1="-21.59" x2="58.5" y2="3.75" width="0" layer="19" extent="16-16"/>
+<wire x1="72.39" y1="31.75" x2="58.5" y2="3.75" width="0" layer="19" extent="16-16"/>
 </signal>
 <signal name="N$39">
 <contactref element="X1" pad="A50"/>
 <contactref element="U$2" pad="P$192"/>
-<wire x1="27.94" y1="-24.13" x2="59.5" y2="3.75" width="0" layer="19" extent="16-16"/>
+<wire x1="74.93" y1="34.29" x2="59.5" y2="3.75" width="0" layer="19" extent="16-16"/>
 </signal>
 <signal name="N$40">
 <contactref element="X1" pad="A51"/>
 <contactref element="U$2" pad="P$208"/>
-<wire x1="30.48" y1="-21.59" x2="60.5" y2="3.75" width="0" layer="19" extent="16-16"/>
+<wire x1="77.47" y1="31.75" x2="60.5" y2="3.75" width="0" layer="19" extent="16-16"/>
 </signal>
 <signal name="N$41">
 <contactref element="X1" pad="A52"/>
 <contactref element="U$2" pad="P$224"/>
-<wire x1="33.02" y1="-24.13" x2="61.5" y2="3.75" width="0" layer="19" extent="16-16"/>
+<wire x1="80.01" y1="34.29" x2="61.5" y2="3.75" width="0" layer="19" extent="16-16"/>
 </signal>
 <signal name="N$42">
 <contactref element="X1" pad="A53"/>
 <contactref element="U$2" pad="P$240"/>
-<wire x1="35.56" y1="-21.59" x2="62.5" y2="3.75" width="0" layer="19" extent="16-16"/>
+<wire x1="82.55" y1="31.75" x2="62.5" y2="3.75" width="0" layer="19" extent="16-16"/>
 </signal>
 <signal name="N$43">
 <contactref element="X1" pad="A54"/>
 <contactref element="U$2" pad="P$256"/>
-<wire x1="38.1" y1="-24.13" x2="63.5" y2="3.75" width="0" layer="19" extent="16-16"/>
+<wire x1="85.09" y1="34.29" x2="63.5" y2="3.75" width="0" layer="19" extent="16-16"/>
 </signal>
 </signals>

Commit message: re-routed wires so i could stop f***ing getting mixed up on orientation
Connections:
- net N$29: now also U$2.P$225, X1.A54; no longer U$2.P$32, X1.A40
- net N$30: now also U$2.P$233, X1.A53; no longer U$2.P$48, X1.A41
- net N$31: now also U$2.P$193, X1.A52; no longer U$2.P$64, X1.A42
- net N$32: now also U$2.P$201, X1.A51; no longer U$2.P$80, X1.A43
- net N$33: now also U$2.P$161, X1.A50; no longer U$2.P$96, X1.A44
- net N$34: now also U$2.P$169, X1.A49; no longer U$2.P$112, X1.A45
- net N$35: now also U$2.P$129, X1.A48; no longer U$2.P$128, X1.A46
- net N$36: now also U$2.P$137; no longer U$2.P$144
- net N$37: now also U$2.P$97, X1.A46; no longer U$2.P$160, X1.A48
- net N$38: now also U$2.P$105, X1.A45; no longer U$2.P$176, X1.A49
- net N$39: now also U$2.P$65, X1.A44; no longer U$2.P$192, X1.A50
- net N$40: now also U$2.P$73, X1.A43; no longer U$2.P$208, X1.A51
- net N$41: now also U$2.P$33, X1.A42; no longer U$2.P$224, X1.A52
- net N$42: now also U$2.P$41, X1.A41; no longer U$2.P$240, X1.A53
- net N$43: now also U$2.P$17, X1.A40; no longer U$2.P$256, X1.A54
Changed lines of the file:
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@@
 </signal>
 <signal name="N$29">
-<contactref element="X1" pad="A40"/>
-<contactref element="U$2" pad="P$32"/>
-<wire x1="49.53" y1="34.29" x2="49.5" y2="3.75" width="0" layer="19" extent="16-16"/>
+<contactref element="U$2" pad="P$225"/>
+<contactref element="X1" pad="A54"/>
+<wire x1="63.5" y1="3.75" x2="85.09" y2="13.97" width="0" layer="19" extent="16-16"/>
 </signal>
 <signal name="N$30">
-<contactref element="X1" pad="A41"/>
-<contactref element="U$2" pad="P$48"/>
-<wire x1="52.07" y1="31.75" x2="50.5" y2="3.75" width="0" layer="19" extent="16-16"/>
+<contactref element="U$2" pad="P$233"/>
+<contactref element="X1" pad="A53"/>
+<wire x1="62.5" y1="3.75" x2="82.55" y2="13.97" width="0" layer="19" extent="16-16"/>
 </signal>
 <signal name="N$31">
-<contactref element="X1" pad="A42"/>
-<contactref element="U$2" pad="P$64"/>
-<wire x1="54.61" y1="34.29" x2="51.5" y2="3.75" width="0" layer="19" extent="16-16"/>
+<contactref element="U$2" pad="P$193"/>
+<contactref element="X1" pad="A52"/>
+<wire x1="61.5" y1="3.75" x2="80.01" y2="13.97" width="0" layer="19" extent="16-16"/>
 </signal>
 <signal name="N$32">
-<contactref element="X1" pad="A43"/>
-<contactref element="U$2" pad="P$80"/>
-<wire x1="57.15" y1="31.75" x2="52.5" y2="3.75" width="0" layer="19" extent="16-16"/>
+<contactref element="U$2" pad="P$201"/>
+<contactref element="X1" pad="A51"/>
+<wire x1="60.5" y1="3.75" x2="77.47" y2="13.97" width="0" layer="19" extent="16-16"/>
 </signal>
 <signal name="N$33">
-<contactref element="X1" pad="A44"/>
-<contactref element="U$2" pad="P$96"/>
-<wire x1="59.69" y1="34.29" x2="53.5" y2="3.75" width="0" layer="19" extent="16-16"/>
+<contactref element="U$2" pad="P$161"/>
+<contactref element="X1" pad="A50"/>
+<wire x1="59.5" y1="3.75" x2="74.93" y2="13.97" width="0" layer="19" extent="16-16"/>
 </signal>
 <signal name="N$34">
-<contactref element="X1" pad="A45"/>
-<contactref element="U$2" pad="P$112"/>
-<wire x1="62.23" y1="31.75" x2="54.5" y2="3.75" width="0" layer="19" extent="16-16"/>
+<contactref element="U$2" pad="P$169"/>
+<contactref element="X1" pad="A49"/>
+<wire x1="58.5" y1="3.75" x2="72.39" y2="13.97" width="0" layer="19" extent="16-16"/>
 </signal>
 <signal name="N$35">
-<contactref element="X1" pad="A46"/>
-<contactref element="U$2" pad="P$128"/>
-<wire x1="64.77" y1="34.29" x2="55.5" y2="3.75" width="0" layer="19" extent="16-16"/>
+<contactref element="U$2" pad="P$129"/>
+<contactref element="X1" pad="A48"/>
+<wire x1="57.5" y1="3.75" x2="69.85" y2="13.97" width="0" layer="19" extent="16-16"/>
 </signal>
 <signal name="N$36">
+<contactref element="U$2" pad="P$137"/>
 <contactref element="X1" pad="A47"/>
-<contactref element="U$2" pad="P$144"/>
-<wire x1="67.31" y1="31.75" x2="56.5" y2="3.75" width="0" layer="19" extent="16-16"/>
+<wire x1="56.5" y1="3.75" x2="67.31" y2="13.97" width="0" layer="19" extent="16-16"/>
 </signal>
 <signal name="N$37">
-<contactref element="X1" pad="A48"/>
-<contactref element="U$2" pad="P$160"/>
-<wire x1="69.85" y1="34.29" x2="57.5" y2="3.75" width="0" layer="19" extent="16-16"/>
+<contactref element="U$2" pad="P$97"/>
+<contactref element="X1" pad="A46"/>
+<wire x1="55.5" y1="3.75" x2="64.77" y2="13.97" width="0" layer="19" extent="16-16"/>
 </signal>
 <signal name="N$38">
-<contactref element="X1" pad="A49"/>
-<contactref element="U$2" pad="P$176"/>
-<wire x1="72.39" y1="31.75" x2="58.5" y2="3.75" width="0" layer="19" extent="16-16"/>
+<contactref element="U$2" pad="P$105"/>
+<contactref element="X1" pad="A45"/>
+<wire x1="54.5" y1="3.75" x2="62.23" y2="13.97" width="0" layer="19" extent="16-16"/>
 </signal>
 <signal name="N$39">
-<contactref element="X1" pad="A50"/>
-<contactref element="U$2" pad="P$192"/>
-<wire x1="74.93" y1="34.29" x2="59.5" y2="3.75" width="0" layer="19" extent="16-16"/>
+<contactref element="U$2" pad="P$65"/>
+<contactref element="X1" pad="A44"/>
+<wire x1="53.5" y1="3.75" x2="59.69" y2="13.97" width="0" layer="19" extent="16-16"/>
 </signal>
 <signal name="N$40">
-<contactref element="X1" pad="A51"/>
-<contactref element="U$2" pad="P$208"/>
-<wire x1="77.47" y1="31.75" x2="60.5" y2="3.75" width="0" layer="19" extent="16-16"/>
+<contactref element="U$2" pad="P$73"/>
+<contactref element="X1" pad="A43"/>
+<wire x1="52.5" y1="3.75" x2="57.15" y2="13.97" width="0" layer="19" extent="16-16"/>
 </signal>
 <signal name="N$41">
-<contactref element="X1" pad="A52"/>
-<contactref element="U$2" pad="P$224"/>
-<wire x1="80.01" y1="34.29" x2="61.5" y2="3.75" width="0" layer="19" extent="16-16"/>
+<contactref element="U$2" pad="P$33"/>
+<contactref element="X1" pad="A42"/>
+<wire x1="51.5" y1="3.75" x2="54.61" y2="13.97" width="0" layer="19" extent="16-16"/>
 </signal>
 <signal name="N$42">
-<contactref element="X1" pad="A53"/>
-<contactref element="U$2" pad="P$240"/>
-<wire x1="82.55" y1="31.75" x2="62.5" y2="3.75" width="0" layer="19" extent="16-16"/>
+<contactref element="U$2" pad="P$41"/>
+<contactref element="X1" pad="A41"/>
+<wire x1="50.5" y1="3.75" x2="52.07" y2="13.97" width="0" layer="19" extent="16-16"/>
 </signal>
 <signal name="N$43">
-<contactref element="X1" pad="A54"/>
-<contactref element="U$2" pad="P$256"/>
-<wire x1="85.09" y1="34.29" x2="63.5" y2="3.75" width="0" layer="19" extent="16-16"/>
+<contactref element="U$2" pad="P$17"/>
+<contactref element="X1" pad="A40"/>
+<wire x1="49.5" y1="3.75" x2="49.53" y2="13.97" width="0" layer="19" extent="16-16"/>
 </signal>
 </signals>
