File: GPIO_board/gpio_board.brd (EAGLE design)
At the start: 93.6 x 79 mm, 15 parts, among them J1 SWITCHES, J2 LED1, J3 LED2, Q1 IRF520, Q2 IRF520, Q3 IRF520, X1 PCI-E-164SLOT

Commit message: added ground pad to proto grid
Connections:
- removed net N$29: U$2.P$225, X1.A68
- net GND: now also U$2.P$225, X1.A68
Routing:
- net N$29: track 13.4 -> 0.00 mm
- net GND: track 76.1 -> 89.5 mm
Changed lines of the file:
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@@
 <vertex x="-1.27" y="11.43"/>
 </polygon>
+<contactref element="U$2" pad="P$225"/>
+<contactref element="X1" pad="A68"/>
+<wire x1="77.5" y1="3.75" x2="77.5" y2="6.38" width="0.4064" layer="16"/>
+<wire x1="77.5" y1="6.38" x2="85.09" y2="13.97" width="0.4064" layer="16"/>
 </signal>
 <signal name="N$1">
@@
 <wire x1="44.45" y1="11.43" x2="46.99" y2="13.97" width="0.4064" layer="1"/>
 </signal>
-<signal name="N$29">
-<contactref element="U$2" pad="P$225"/>
-<contactref element="X1" pad="A68"/>
-<wire x1="77.5" y1="3.75" x2="77.5" y2="6.38" width="0.4064" layer="16"/>
-<wire x1="77.5" y1="6.38" x2="85.09" y2="13.97" width="0.4064" layer="16"/>
-</signal>
 <signal name="N$30">
 <contactref element="U$2" pad="P$233"/>
@@
 <wire x1="51.562" y1="3.812" x2="51.5" y2="3.75" width="0.4064" layer="16"/>
 </signal>
-<signal name="N$43">
+<signal name="N$43" class="1">
 <contactref element="U$2" pad="P$17"/>
 <contactref element="X1" pad="A40"/>

Commit message: added headers for VIN and serial port. fixed issues with redundant manual route to ground from pin 1 on teensy.
Parts:
- added J4, J5: (no value), SparkFun-Connectors:1X02
Connections:
- removed net VIN: U$1.VIN
- new net N$29: J4.1, U$1.0
- new net N$44: J4.2, U$1.1
- new net N$45: J5.2, U$1.VIN
- net GND: now also J5.1
Routing:
- net GND: track 89.5 -> 50.3 mm, vias 2 -> 0
- net N$45: track 0.00 -> 37.6 mm
- net N$44: track 0.00 -> 21.1 mm
- net N$29: track 0.00 -> 19.0 mm
- net N$3: track 0.00 -> 3.81 mm
- net N$2: track 0.00 -> 3.81 mm
- net N$1: track 0.00 -> 3.81 mm
Changed lines of the file:
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@@
 <setting verticaltext="up"/>
 </settings>
-<grid distance="0.01" unitdist="inch" unit="inch" style="lines" multiple="1" display="yes" altdistance="0.005" altunitdist="inch" altunit="inch"/>
+<grid distance="0.01" unitdist="inch" unit="inch" style="lines" multiple="1" display="no" altdistance="0.005" altunitdist="inch" altunit="inch"/>
 <layers>
 <layer number="1" name="Top" color="4" fill="1" visible="yes" active="yes"/>
@@
 <element name="X1" library="con-pc" package="PCI-E_SLOT" value="PCI-E-164SLOT" x="0" y="0"/>
 <element name="U$2" library="talon_lbr" package="PROTO_GRID16" value="PROTO_GRID" x="46.99" y="52.07" rot="MR180"/>
+<element name="J4" library="SparkFun-Connectors" package="1X02" value="" x="21.59" y="65.786"/>
+<element name="J5" library="SparkFun-Connectors" package="1X02" value="" x="66.294" y="61.722"/>
 </elements>
 <signals>
-<signal name="VIN">
-<contactref element="U$1" pad="VIN"/>
-</signal>
-<signal name="GND" class="1">
+<signal name="GND">
 <contactref element="U$1" pad="GND"/>
 <contactref element="U$1" pad="AGND"/>
@@
 <contactref element="X1" pad="A8"/>
 <polygon width="0.4064" layer="16">
-<vertex x="-1.27" y="82.55"/>
 <vertex x="-1.27" y="13.97"/>
 <vertex x="8.89" y="13.97"/>
@@
 <vertex x="-1.27" y="83.82"/>
 </polygon>
-<wire x1="18.5" y1="3.75" x2="18.5" y2="12.7" width="0.4064" layer="16"/>
-<wire x1="18.5" y1="12.7" x2="18.5" y2="27.22" width="0.4064" layer="16"/>
-<wire x1="18.5" y1="27.22" x2="15.24" y2="30.48" width="0.4064" layer="16"/>
-<wire x1="15.24" y1="30.48" x2="15.24" y2="43.18" width="0.4064" layer="16"/>
-<via x="15.24" y="43.18" extent="1-16" drill="0.508"/>
-<wire x1="15.24" y1="43.18" x2="15.24" y2="44.45" width="0.4064" layer="1"/>
-<wire x1="15.24" y1="44.45" x2="17.78" y2="46.99" width="0.4064" layer="1"/>
-<via x="17.78" y="46.99" extent="1-16" drill="0.508"/>
-<wire x1="17.78" y1="46.99" x2="21.59" y2="50.8" width="0.4064" layer="16"/>
-<wire x1="17.5" y1="3.75" x2="17.5" y2="11.7" width="0.4064" layer="16"/>
-<wire x1="17.5" y1="11.7" x2="18.5" y2="12.7" width="0.4064" layer="16"/>
-<wire x1="16.5" y1="3.75" x2="16.5" y2="10.7" width="0.4064" layer="16"/>
-<wire x1="16.5" y1="10.7" x2="17.5" y2="11.7" width="0.4064" layer="16"/>
-<wire x1="15.5" y1="3.75" x2="15.5" y2="9.7" width="0.4064" layer="16"/>
-<wire x1="15.5" y1="9.7" x2="16.5" y2="10.7" width="0.4064" layer="16"/>
 <polygon width="0.4064" layer="1">
 <vertex x="-1.27" y="83.82"/>
@@
 <wire x1="77.5" y1="3.75" x2="77.5" y2="6.38" width="0.4064" layer="16"/>
 <wire x1="77.5" y1="6.38" x2="85.09" y2="13.97" width="0.4064" layer="16"/>
+<contactref element="J5" pad="1"/>
+<wire x1="18.5" y1="3.75" x2="18.5" y2="12.192" width="0.4064" layer="16"/>
+<wire x1="18.5" y1="12.192" x2="18.5" y2="12.404" width="0.4064" layer="16"/>
+<wire x1="18.5" y1="12.404" x2="18.542" y2="12.446" width="0.4064" layer="16"/>
+<wire x1="17.5" y1="3.75" x2="17.5" y2="11.404" width="0.4064" layer="16"/>
+<wire x1="17.5" y1="11.404" x2="18.5" y2="12.404" width="0.4064" layer="16"/>
+<wire x1="16.5" y1="3.75" x2="16.5" y2="10.192" width="0.4064" layer="16"/>
+<wire x1="16.5" y1="10.192" x2="18.5" y2="12.192" width="0.4064" layer="16"/>
+<wire x1="15.5" y1="3.75" x2="15.5" y2="9.404" width="0.4064" layer="16"/>
+<wire x1="15.5" y1="9.404" x2="18.5" y2="12.404" width="0.4064" layer="16"/>
 </signal>
 <signal name="N$1">
 <contactref element="R1" pad="P$2"/>
 <contactref element="Q1" pad="G"/>
-<wire x1="55.88" y1="66.04" x2="55.88" y2="69.85" width="0" layer="19" extent="1-1"/>
+<wire x1="55.88" y1="69.85" x2="55.88" y2="66.04" width="0.4064" layer="1"/>
 </signal>
 <signal name="N$2">
 <contactref element="R2" pad="P$2"/>
 <contactref element="Q2" pad="G"/>
-<wire x1="44.45" y1="66.04" x2="44.45" y2="69.85" width="0" layer="19" extent="1-1"/>
+<wire x1="44.45" y1="69.85" x2="44.45" y2="66.04" width="0.4064" layer="1"/>
 </signal>
 <signal name="N$3">
 <contactref element="R3" pad="P$2"/>
 <contactref element="Q3" pad="G"/>
-<wire x1="31.75" y1="66.04" x2="31.75" y2="69.85" width="0" layer="19" extent="1-1"/>
+<wire x1="31.75" y1="69.85" x2="31.75" y2="66.04" width="0.4064" layer="1"/>
 </signal>
 <signal name="N$4">
@@
 <wire x1="49.53" y1="3.78" x2="49.5" y2="3.75" width="0.4064" layer="16"/>
 </signal>
+<signal name="N$29">
+<contactref element="U$1" pad="0"/>
+<contactref element="J4" pad="1"/>
+<wire x1="21.59" y1="48.26" x2="23.368" y2="50.038" width="0.4064" layer="1"/>
+<wire x1="23.368" y1="50.038" x2="23.368" y2="61.214" width="0.4064" layer="1"/>
+<wire x1="23.368" y1="61.214" x2="21.59" y2="62.992" width="0.4064" layer="1"/>
+<wire x1="21.59" y1="62.992" x2="21.59" y2="65.786" width="0.4064" layer="1"/>
+</signal>
+<signal name="N$44">
+<contactref element="J4" pad="2"/>
+<contactref element="U$1" pad="1"/>
+<wire x1="21.59" y1="45.72" x2="21.59" y2="45.974" width="0.4064" layer="1"/>
+<wire x1="21.59" y1="45.974" x2="24.13" y2="48.514" width="0.4064" layer="1"/>
+<wire x1="24.13" y1="48.514" x2="24.13" y2="65.786" width="0.4064" layer="1"/>
+</signal>
+<signal name="N$45">
+<contactref element="J5" pad="2"/>
+<contactref element="U$1" pad="VIN"/>
+<wire x1="36.83" y1="50.8" x2="36.83" y2="52.578" width="0.4064" layer="1"/>
+<wire x1="36.83" y1="52.578" x2="38.608" y2="54.356" width="0.4064" layer="1"/>
+<wire x1="38.608" y1="54.356" x2="61.468" y2="54.356" width="0.4064" layer="1"/>
+<wire x1="61.468" y1="54.356" x2="68.834" y2="61.722" width="0.4064" layer="1"/>
+</signal>
 </signals>
